Commit message: [description] laser_filter 수치 정밀 수정, camera, lidar 위치 수정

File: src/omo_r1-ros2/omo_r1_description/urdf/omo_r1.urdf (robot description, URDF)
Before this commit: robot omo_r1, 11 links, 10 joints
Joints:
- joint camera_joint: origin xyz=0.07 0.0 0.63 rpy=0 0.7 0 -> xyz=0.095 0.0 0.375 rpy=0 0 0
- joint imu_joint: origin xyz=0.0 0 0.190 rpy=0 0 1.5758 -> xyz=0.1 0 0.375 rpy=0 0 1.5758
- joint scan_joint: origin xyz=0.06 0 0.230 rpy=0.0 0 3.14159 -> xyz=0.08 0 0.41 rpy=0.0 0 3.14159
